Commit message: added arms

File: automi_description/urdf/arm.urdf.xacro (robot description, xacro)
@@ -1,3 +1,83 @@
 <?xml version="1.0"?>
 <robot xmlns:xacro="http://www.ros.org/wiki/xacro">
+    <xacro:macro name="arm" params="name parent *origin reflect">
+        <xacro:AX12
+            name="${name}_shoulder_pitch"
+            parent="${parent}"
+            child="${name}_shoulder">
+            <xacro:insert_block name="origin"/>
+            <origin xyz="0.0 0.0 0.04" rpy="0.0 0.0 0.0"/>
+        </xacro:AX12>
+        <link name="${name}_shoulder">
+            <inertial>
+                <origin xyz="0.0 0.0 0.0" rpy="0.0 0.0 0.0"/>
+                <mass value="1.0"/>
+                <inertia ixx="0.0" ixy="0.0" ixz="0.0" iyy="0.0" iyz="0.0" izz="0.0"/>
+            </inertial>
+            <visual name="">
+                <origin xyz="0.0 0.0 0.0" rpy="0.0 0.0 0.0"/>
+                <geometry>
+                    <box size="0.04 0.04 0.03"/>
+                </geometry>
+            </visual>
+            <collision>
+                <origin xyz="0.0 0.0 0.0" rpy="0.0 0.0 0.0"/>
+                <geometry>
+                    <box size="0.04 0.04 0.03"/>
+                </geometry>
+            </collision>
+        </link>
+        <xacro:AX12
+            name="${name}_shoulder_roll"
+            parent="${name}_shoulder"
+            child="${name}_arm">
+            <origin xyz="0.0 0.05 0.0" rpy="0.0 ${reflect*PI/2} 0.0"/>
+            <origin xyz="0.0 0.0 0.0" rpy="0.0 0.0 0.0"/>
+        </xacro:AX12>
+        <link name="${name}_arm">
+            <inertial>
+                <origin xyz="0.0 0.0 0.0" rpy="0.0 0.0 0.0"/>
+                <mass value="1.0"/>
+                <inertia ixx="0.0" ixy="0.0" ixz="0.0" iyy="0.0" iyz="0.0" izz="0.0"/>
+            </inertial>
+            <visual name="">
+                <origin xyz="0.0 0.05 0.0" rpy="0.0 0.0 0.0"/>
+                <geometry>
+                    <box size="0.02 0.1 0.02"/>
+                </geometry>
+            </visual>
+            <collision>
+                <origin xyz="0.0 0.05 0.0" rpy="0.0 0.0 0.0"/>
+                <geometry>
+                    <box size="0.02 0.1 0.02"/>
+                </geometry>
+            </collision>
+        </link>
+        <xacro:AX12
+            name="${name}_elbow"
+            parent="${name}_arm"
+            child="${name}_gripper">
+            <origin xyz="0.0 0.1 0.0" rpy="0.0 ${-reflect*PI/2} 0.0"/>
+            <origin xyz="0.0 0.0 0.0" rpy="0.0 0.0 0.0"/>
+        </xacro:AX12>
+        <link name="${name}_gripper">
+            <inertial>
+                <origin xyz="0.0 0.0 0.0" rpy="0.0 0.0 0.0"/>
+                <mass value="1.0"/>
+                <inertia ixx="0.0" ixy="0.0" ixz="0.0" iyy="0.0" iyz="0.0" izz="0.0"/>
+            </inertial>
+            <visual name="">
+                <origin xyz="0.0 0.05 0.0" rpy="0.0 0.0 0.0"/>
+                <geometry>
+                    <box size="0.02 0.1 0.02"/>
+                </geometry>
+            </visual>
+            <collision>
+                <origin xyz="0.0 0.05 0.0" rpy="0.0 0.0 0.0"/>
+                <geometry>
+                    <box size="0.02 0.1 0.02"/>
+                </geometry>
+            </collision>
+        </link>
+    </xacro:macro>
 </robot>

File: automi_description/urdf/automi.urdf.xacro (robot description, xacro)
@@ -4,5 +4,5 @@
     <xacro:include filename="$(find automi_description)/urdf/dynamixels.urdf.xacro" />
     <!-- <xacro:include filename="$(find automi_description)/urdf/torso.urdf.xacro" /> -->
-    <!-- <xacro:include filename="$(find automi_description)/urdf/arm.urdf.xacro" /> -->
+    <xacro:include filename="$(find automi_description)/urdf/arm.urdf.xacro" />
     <xacro:include filename="$(find automi_description)/urdf/leg.urdf.xacro" />
     <link name="1">
@@ -28,5 +28,5 @@
         parent="1"
         reflect="1">
-        <origin xyz="0.1 0.0 0.0" rpy="0.0 ${PI} 0.0"/>
+        <origin xyz="0.075 0.0 0.0" rpy="0.0 ${PI} 0.0"/>
     </xacro:leg>
     <xacro:leg
@@ -34,5 +34,17 @@
         parent="1"
         reflect="-1">
-        <origin xyz="-0.1 0.0 0.0" rpy="0.0 ${PI} 0.0"/>
+        <origin xyz="-0.075 0.0 0.0" rpy="0.0 ${PI} 0.0"/>
     </xacro:leg>
+    <xacro:arm
+        name="right"
+        parent="1"
+        reflect="-1">
+        <origin xyz="-0.1 0.0 0.2" rpy="${3*PI/2} 0.0 ${PI/2}"/>
+    </xacro:arm>
+    <xacro:arm
+        name="left"
+        parent="1"
+        reflect="1">
+        <origin xyz="0.1 0.0 0.2" rpy="${3*PI/2} 0.0 ${-PI/2}"/>
+    </xacro:arm>
 </robot>

File: automi_description/urdf/leg.urdf.xacro (robot description, xacro)
@@ -19,5 +19,5 @@
                 <origin xyz="0.0 0.0 0.04" rpy="0.0 0.0 ${PI/2}"/>
                 <geometry>
-                    <box size="0.15 0.05 0.005"/>
+                    <box size="0.10 0.05 0.005"/>
                 </geometry>
             </collision>
@@ -25,5 +25,5 @@
                 <origin xyz="0.0 0.0 0.04" rpy="0.0 0.0 ${PI/2}"/>
                 <geometry>
-                    <box size="0.15 0.05 0.005"/>
+                    <box size="0.10 0.05 0.005"/>
                 </geometry>
             </visual>
@@ -47,5 +47,5 @@
             parent="${name}_int_hip"
             child="${name}_upper_leg">
-            <origin xyz="0.0 0.0 0.0" rpy="0.0 0.0 0.0"/>
+            <origin xyz="0.0 0.0 0.0" rpy="0.0 ${PI/2*(1+reflect)} 0.0"/>
             <origin xyz="0.0 0.0 0.0" rpy="${PI/2} 0.0 ${PI/2}"/>
         </xacro:MX64>
@@ -99,5 +99,5 @@
             parent="${name}_lower_leg"
             child="${name}_int_ankle">
-            <origin xyz="0.0 -0.15 0.0" rpy="0.0 ${PI} 0"/>
+            <origin xyz="0.0 -0.15 0.0" rpy="0.0 0 0"/>
             <origin xyz="0.0 0.0 0.0" rpy="0.0 0.0 0.0"/>
         </xacro:MX28>
@@ -113,6 +113,6 @@
             parent="${name}_int_ankle"
             child="${name}_foot">
-            <origin xyz="0.05 0.0 0.0" rpy="0 0 0"/>
-            <origin xyz="-0.03 -0.03 0.0" rpy="0 ${PI/2} 0.0"/>
+            <origin xyz="${reflect*0.05} 0.0 0.0" rpy="0 0 0"/>
+            <origin xyz="${-reflect*0.03} -0.03 0.0" rpy="0 ${reflect*-PI/2} 0.0"/>
         </xacro:MX64>
         <link name="${name}_foot">

Commit message: added torso and transmissions

File: automi_description/urdf/arm.urdf.xacro (robot description, xacro)
@@ -3,5 +3,5 @@
     <xacro:macro name="arm" params="name parent *origin reflect">
         <xacro:AX12
-            name="${name}_shoulder_pitch"
+            name="${name}_shoulder_p"
             parent="${parent}"
             child="${name}_shoulder">
@@ -29,5 +29,5 @@
         </link>
         <xacro:AX12
-            name="${name}_shoulder_roll"
+            name="${name}_shoulder_r"
             parent="${name}_shoulder"
             child="${name}_arm">

File: automi_description/urdf/automi.urdf.xacro (robot description, xacro)
@@ -3,48 +3,100 @@
     <xacro:property name="PI" value="3.1415926535897931"/>
     <xacro:include filename="$(find automi_description)/urdf/dynamixels.urdf.xacro" />
-    <!-- <xacro:include filename="$(find automi_description)/urdf/torso.urdf.xacro" /> -->
+    <xacro:include filename="$(find automi_description)/urdf/torso.urdf.xacro" />
     <xacro:include filename="$(find automi_description)/urdf/arm.urdf.xacro" />
     <xacro:include filename="$(find automi_description)/urdf/leg.urdf.xacro" />
-    <link name="1">
+    <link name="floating_base">
         <inertial>
-            <origin xyz="0.0 0.0 0.0" rpy="0.0 0.0 0.0"/>
-            <mass value="1.0"/>
-            <inertia ixx="0.0" ixy="0.0" ixz="0.0" iyy="0.0" iyz="0.0" izz="0.0"/>
+            <mass value="0.0005"/>
         </inertial>
-        <collision>
-            <origin xyz="0.0 0.0 0.0" rpy="0.0 0.0 0.0"/>
-            <geometry>
-                <box size="0.1 0.05 0.05"/>
-            </geometry>
-        </collision>
-        <visual>
-            <geometry>
-                <box size="0.1 0.05 0.05"/>
-            </geometry>
-        </visual>
     </link>
+    <xacro:torso
+        name="body"
+        parent="floating_base">
+        <origin xyz="0.0 0.0 0.0" rpy="0.0 0.0 0.0"/>
+    </xacro:torso>
     <xacro:leg
-        name="left"
-        parent="1"
+        name="l"
+        parent="body_hip"
         reflect="1">
         <origin xyz="0.075 0.0 0.0" rpy="0.0 ${PI} 0.0"/>
     </xacro:leg>
     <xacro:leg
-        name="right"
-        parent="1"
+        name="r"
+        parent="body_hip"
         reflect="-1">
         <origin xyz="-0.075 0.0 0.0" rpy="0.0 ${PI} 0.0"/>
     </xacro:leg>
     <xacro:arm
-        name="right"
-        parent="1"
+        name="r"
+        parent="body_chest"
         reflect="-1">
-        <origin xyz="-0.1 0.0 0.2" rpy="${3*PI/2} 0.0 ${PI/2}"/>
+        <origin xyz="-0.1 0.0 0.05" rpy="${3*PI/2} 0.0 ${PI/2}"/>
     </xacro:arm>
     <xacro:arm
-        name="left"
-        parent="1"
+        name="l"
+        parent="body_chest"
         reflect="1">
-        <origin xyz="0.1 0.0 0.2" rpy="${3*PI/2} 0.0 ${-PI/2}"/>
+        <origin xyz="0.1 0.0 0.05" rpy="${3*PI/2} 0.0 ${-PI/2}"/>
     </xacro:arm>
+    <gazebo>
+        <plugin name="joint_state_publisher" filename="libgazebo_ros_joint_state_publisher.so">
+            <jointName>
+                head_pan    ,
+                head_tilt   ,
+                r_hip_r     ,
+                r_hip_p     ,
+                r_hip_y     ,
+                r_knee      ,
+                r_ankle_r   ,
+                r_ankle_p   ,
+                r_shoulder_r,
+                r_shoulder_p,
+                r_elbow     ,
+                l_hip_r     ,
+                l_hip_p     ,
+                l_hip_y     ,
+                l_knee      ,
+                l_ankle_r   ,
+                l_ankle_p   ,
+                l_shoulder_r,
+                l_shoulder_p,
+                l_elbow
+            </jointName>
+            <updateRate>60.0</updateRate>
+            <alwaysOn>true</alwaysOn>
+        </plugin>
+    </gazebo>
+    <xacro:macro name="trans" params="num joint">
+        <transmission name="tran${num}">
+        <joint name="${joint}">
+            <hardwareInterface>hardware_interface/PositionJointInterface</hardwareInterface>
+        </joint>
+        <type>transmission_interface/SimpleTransmission</type>
+        <actuator name="servo${num}">
+            <hardwareInterface>hardware_interface/PositionJointInterface</hardwareInterface>
+            <mechanicalReduction>1</mechanicalReduction>
+        </actuator>
+        </transmission>
+    </xacro:macro>
+    <xacro:trans num="1"  joint="r_hip_r"/>
+    <xacro:trans num="2"  joint="r_hip_p"/>
+    <xacro:trans num="3"  joint="r_hip_y"/>
+    <xacro:trans num="4"  joint="r_knee"/>
+    <xacro:trans num="5"  joint="r_ankle_r"/>
+    <xacro:trans num="6"  joint="r_ankle_p"/>
+    <xacro:trans num="7" joint="l_hip_r"/>
+    <xacro:trans num="8" joint="l_hip_p"/>
+    <xacro:trans num="9" joint="l_hip_y"/>
+    <xacro:trans num="10" joint="l_knee"/>
+    <xacro:trans num="11" joint="l_ankle_r"/>
+    <xacro:trans num="12" joint="l_ankle_p"/>
+    <xacro:trans num="13"  joint="r_shoulder_r"/>
+    <xacro:trans num="14" joint="r_shoulder_p"/>
+    <xacro:trans num="15" joint="r_elbow"/>
+    <xacro:trans num="16" joint="l_shoulder_r"/>
+    <xacro:trans num="17" joint="l_shoulder_p"/>
+    <xacro:trans num="18" joint="l_elbow"/>
+    <xacro:trans num="19"  joint="head_pan"/>
+    <xacro:trans num="20"  joint="head_tilt"/>
 </robot>

File: automi_description/urdf/leg.urdf.xacro (robot description, xacro)
@@ -4,5 +4,5 @@
         <!-- LINKS -->
         <xacro:AX12
-            name="${name}_hip_yaw"
+            name="${name}_hip_y"
             parent="${parent}"
             child="${name}_top_Ubar">
@@ -30,5 +30,5 @@
         </link>
         <xacro:MX28
-            name="${name}_hip_roll"
+            name="${name}_hip_r"
             parent="${name}_top_Ubar"
             child="${name}_int_hip">
@@ -44,5 +44,5 @@
         </link>
         <xacro:MX64
-            name="${name}_hip_pitch"
+            name="${name}_hip_p"
             parent="${name}_int_hip"
             child="${name}_upper_leg">
@@ -96,5 +96,5 @@
         </link>
         <xacro:MX28
-            name="${name}_ankle_pitch"
+            name="${name}_ankle_p"
             parent="${name}_lower_leg"
             child="${name}_int_ankle">
@@ -110,9 +110,9 @@
         </link>
         <xacro:MX64
-            name="${name}_ankle_roll"
+            name="${name}_ankle_r"
             parent="${name}_int_ankle"
             child="${name}_foot">
             <origin xyz="${reflect*0.05} 0.0 0.0" rpy="0 0 0"/>
-            <origin xyz="${-reflect*0.03} -0.03 0.0" rpy="0 ${reflect*-PI/2} 0.0"/>
+            <origin xyz="0.0 0.0 0.0" rpy="0 ${reflect*-PI/2} 0.0"/>
         </xacro:MX64>
         <link name="${name}_foot">
@@ -123,5 +123,5 @@
             </inertial>
             <visual name="">
-                <origin xyz="0.0 0.0 0.0" rpy="0.0 0.0 0.0"/>
+                <origin xyz="0.0 -0.04 0.04" rpy="0.0 0.0 0.0"/>
                 <geometry>
                     <box size="0.10 0.005 0.14"/>
@@ -129,5 +129,5 @@
             </visual>
             <collision>
-                <origin xyz="0.0 0.0 0.0" rpy="0.0 0.0 0.0"/>
+                <origin xyz="0.0 -0.04 0.04" rpy="0.0 0.0 0.0"/>
                 <geometry>
                     <box size="0.10 0.005 0.14"/>

File: automi_description/urdf/torso.urdf.xacro (robot description, xacro)
@@ -1,3 +1,131 @@
 <?xml version="1.0"?>
 <robot xmlns:xacro="http://www.ros.org/wiki/xacro">
+    <xacro:macro name="torso" params="name parent *origin">
+        <joint name="${name}_waist" type="fixed">
+            <xacro:insert_block name="origin"/>
+            <parent link="${parent}"/>
+            <child link="${name}_hip"/>
+        </joint>
+        <gazebo reference="${name}_waist">
+			<provideFeedback>true</provideFeedback>
+            <preserveFixedJoint>true</preserveFixedJoint>
+		</gazebo>
+        <link name="${name}_hip">
+            <inertial>
+                <origin xyz="0.0 0.0 0.0" rpy="0.0 0.0 0.0"/>
+                <mass value="1.0"/>
+                <inertia ixx="0.0" ixy="0.0" ixz="0.0" iyy="0.0" iyz="0.0" izz="0.0"/>
+            </inertial>
+            <collision>
+                <origin xyz="0.0 0.0 0.0" rpy="0.0 0.0 0.0"/>
+                <geometry>
+                    <box size="0.1 0.05 0.05"/>
+                </geometry>
+            </collision>
+            <visual>
+                <geometry>
+                    <box size="0.1 0.05 0.05"/>
+                </geometry>
+            </visual>
+        </link>
+        <joint name="${name}_core_j" type="fixed">
+        <origin xyz="0.0 0.0 0.075" rpy="0.0 0.0 0.0"/>
+            <parent link="${name}_hip"/>
+            <child link="${name}_core"/>
+        </joint>
+        <gazebo reference="${name}_core_j">
+			<provideFeedback>true</provideFeedback>
+            <preserveFixedJoint>true</preserveFixedJoint>
+		</gazebo>
+        <link name="${name}_core">
+            <inertial>
+                <origin xyz="0.0 0.0 0.0" rpy="0.0 0.0 0.0"/>
+                <mass value="1.0"/>
+                <inertia ixx="0.0" ixy="0.0" ixz="0.0" iyy="0.0" iyz="0.0" izz="0.0"/>
+            </inertial>
+            <visual name="">
+                <origin xyz="0.0 0.0 0.0" rpy="0.0 0.0 0.0"/>
+                <geometry>
+                    <box size="0.075 0.05 0.15"/>
+                </geometry>
+            </visual>
+            <collision>
+                <origin xyz="0.0 0.0 0.0" rpy="0.0 0.0 0.0"/>
+                <geometry>
+                    <box size="0.075 0.05 0.15"/>
+                </geometry>
+            </collision>
+        </link>
+        <joint name="${name}_chest_j" type="fixed">
+            <parent link="${name}_core"/>
+            <child link="${name}_chest"/>
+            <origin xyz="0.0 0.0 0.075" rpy="0.0 0.0 0.0"/>
+        </joint>
+        <gazebo reference="${name}_chest_j">
+			<provideFeedback>true</provideFeedback>
+            <preserveFixedJoint>true</preserveFixedJoint>
+		</gazebo>
+        <link name="${name}_chest">
+            <inertial>
+                <origin xyz="0.0 0.0 0.0" rpy="0.0 0.0 0.0"/>
+                <mass value="1.0"/>
+                <inertia ixx="0.0" ixy="0.0" ixz="0.0" iyy="0.0" iyz="0.0" izz="0.0"/>
+            </inertial>
+            <visual name="">
+                <origin xyz="0.0 0.0 0.0" rpy="0.0 0.0 0.0"/>
+                <geometry>
+                    <box size="0.2 0.05 0.05"/>
+                </geometry>
+            </visual>
+            <collision>
+                <origin xyz="0.0 0.0 0.0" rpy="0.0 0.0 0.0"/>
+                <geometry>
+                    <box size="0.2 0.05 0.05"/>
+                </geometry>
+            </collision>
+        </link>
+        <xacro:AX12
+            name="head_pan"
+            parent="${name}_chest"
+            child="${name}_int_head">
+            <origin xyz="0.0 0.0 0.05" rpy="0.0 0.0 ${PI/2}"/>
+            <origin xyz="0.0 0.0 0.0" rpy="0.0 0.0 0.0"/>
+        </xacro:AX12>
+        <link name="${name}_int_head">
+            <inertial>
+                <mass value="0.0005"/>
+            </inertial>
+        </link>
+        <xacro:AX12
+            name="head_tilt"
+            parent="${name}_int_head"
+            child="${name}_camera_link">
+            <origin xyz="0.0 0.0 0.05" rpy="${PI/2} 0.0 0.0"/>
+            <origin xyz="-0.03 0.0 0.0" rpy="0.0 0.0 0.0"/>
+        </xacro:AX12>
+        <link name="${name}_camera_link">
+            <inertial>
+                <origin xyz="0.0 0.0 0.0" rpy="0.0 0.0 0.0"/>
+                <mass value="1.0"/>
+                <inertia ixx="0.0" ixy="0.0" ixz="0.0" iyy="0.0" iyz="0.0" izz="0.0"/>
+            </inertial>
+            <visual name="">
+                <origin xyz="0.0 0.0 0.0" rpy="0.0 0.0 0.0"/>
+                <geometry>
+                    <box size="0.02 0.02 0.02"/>
+                </geometry>
+            </visual>
+            <collision>
+                <origin xyz="0.0 0.0 0.0" rpy="0.0 0.0 0.0"/>
+                <geometry>
+                    <box size="0.02 0.02 0.02"/>
+                </geometry>
+            </collision>
+        </link>
+        <gazebo reference="${name}_camera_link">
+            <material>
+                Gazebo/Red
+            </material>
+        </gazebo>
+    </xacro:macro>
 </robot>
