Commit message: fixed inertias

File: automi_description/urdf/arm.urdf.xacro (robot description, xacro)
@@ -11,5 +11,5 @@
         <link name="${name}_shoulder">
             <inertial>
-                <origin xyz="0.0 0.0 0.0" rpy="0.0 0.0 0.0"/>
+                <origin xyz="0.0 0.01 0.01" rpy="0.0 0.0 0.0"/>
                 <mass value="0.0114101"/>
                 <inertia ixx="2.20572018e-06" ixy="-0" ixz="-6.183e-11" iyy="4.83772068e-06" iyz="-5.6590326e-07" izz="4.41215019e-06"/>
@@ -37,5 +37,5 @@
         <link name="${name}_arm">
             <inertial>
-                <origin xyz="0.0 0.0 0.0" rpy="0.0 0.0 0.0"/>
+                <origin xyz="0.0 0.07 0.0" rpy="0.0 0.0 0.0"/>
                 <mass value="0.0217184"/>
                 <inertia ixx="8.43192828e-06" ixy="-1.62e-12" ixz="2.16e-12" iyy="8.78536152e-06" iyz="-2.7e-12" izz="1.33461094e-05"/>
@@ -65,5 +65,5 @@
         <link name="${name}_gripper">
             <inertial>
-                <origin xyz="0.0 0.0 0.0" rpy="0.0 0.0 0.0"/>
+                <origin xyz="0.0 0.07 0.0" rpy="0.0 0.0 0.0"/>
                 <mass value="0.0217184"/>
                 <inertia ixx="8.43192828e-06" ixy="-1.62e-12" ixz="2.16e-12" iyy="8.78536152e-06" iyz="-2.7e-12" izz="1.33461094e-05"/>

File: automi_description/urdf/dynamixels.urdf.xacro (robot description, xacro)
@@ -8,5 +8,5 @@
             <axis xyz="0 0 1"/>
             <limit
-                effort="150.0"
+                effort="20.0"
                 velocity="12.0"
                 lower="-2e16"
@@ -28,7 +28,7 @@
         <link name="${name}_AX18">
             <inertial>
-                <origin xyz="0 0 0"/>
-                <mass value="0.115109"/>
-                <inertia ixx="3.3239562e-08" ixy="-1.71315e-12"ixz="7.3197e-12" iyy="1.83264787e-08" iyz="-2.8088019e-10" izz="2.79685224e-08"/>
+                <origin xyz="0 -0.015 0"/>
+                <mass value="0.05590"/>
+                <inertia ixx="0.0000190991666666667" ixy="0" ixz="0" iyy="0.0000122234666666667" iyz="0" izz="0.0000164159666666667"/>
             </inertial>
             <visual>
@@ -58,5 +58,5 @@
             <axis xyz="0 0 1"/>
             <limit
-                effort="150.0"
+                effort="20.0"
                 velocity="12.0"
                 lower="-2e16"
@@ -78,10 +78,10 @@
         <link name="${name}_MX28">
             <inertial>
-                <origin xyz="0 0 0"/>
+                <origin xyz="0 0.01 0"/>
                 <mass value="0.072"/>
                 <inertia
-                    ixx="0" ixy="0" ixz="0"
-                    iyy="0" iyz="0"
-                    izz="0"/>
+                    ixx="0.00002296632" ixy="0" ixz="0"
+                    iyy="0.00001520832" iyz="0"
+                    izz="0.00002296632"/>
             </inertial>
             <visual>
@@ -113,5 +113,5 @@
             <axis xyz="0 0 1"/>
             <limit
-                effort="150.0"
+                effort="20.0"
                 velocity="12.0"
                 lower="-2e16"
@@ -133,10 +133,10 @@
         <link name="${name}_MX64">
             <inertial>
-                <origin xyz="0 0 0"/>
+                <origin xyz="0 0.02 0"/>
                 <mass value="0.1650"/>
                 <inertia
-                    ixx="0" ixy="0" ixz="0"
-                    iyy="0" iyz="0"
-                    izz="0"/>
+                    ixx="0.0000744453875" ixy="0" ixz="0"
+                    iyy="0.0000453343" iyz="0"
+                    izz="0.0000735521875"/>
             </inertial>
             <visual>

File: automi_description/urdf/leg.urdf.xacro (robot description, xacro)
@@ -12,7 +12,7 @@
         <link name="${name}_thigh">
             <inertial>
-                <origin xyz="0.0 0.0 0.0" rpy="0.0 0.0 0.0"/>
+                <origin xyz="0.0 0.01 0.03" rpy="${-PI/2} 0.0 ${PI/2}"/>
                 <mass value="0.0524686"/>
-                <inertia ixx="3.79355686e-05" ixy="1.22736951e-05" ixz="2.4462e-10" iyy="6.47107923e-05" iyz="2.1033e-10" izz="7.72305303e-05"/>
+                <inertia ixx="3.79355686e-05" ixy="1.22736951e-10" ixz="2.4462e-10" iyy="6.47107923e-05" iyz="2.1033e-10" izz="7.72305303e-05"/>
             </inertial>
             <visual name="">
@@ -54,7 +54,7 @@
         <link name="${name}_upper_leg">
             <inertial>
-                <origin xyz="0.0 0.0 0.0" rpy="0.0 0.0 0.0"/>
+                <origin xyz="0.03 0.0 0.0" rpy="${PI/2} 0.0 ${PI/2}"/>
                 <mass value="0.0308695"/>
-                <inertia ixx="2.44928245e-05" ixy="-8.1e-13" ixz="-1.08e-12" iyy="1.5896763e-05" iyz="-1.055808e-07" izz="1.52603879e-05"/>
+                <inertia ixx="2.44928245e-05" ixy="-8.1e-13" ixz="-1.08e-12" iyy="1.5896763e-05" iyz="-1.055808e-10" izz="1.52603879e-05"/>
             </inertial>
             <visual name="">
@@ -82,7 +82,7 @@
         <link name="${name}_lower_leg">
             <inertial>
-                <origin xyz="0.0 0.0 0.0" rpy="0.0 0.0 0.0"/>
+                <origin xyz="0.0 -0.05 0.0" rpy="${PI/2} 0.0 0.0"/>
                 <mass value="0.0387102"/>
-                <inertia ixx="4.41099235e-05" ixy="-0" ixz="-5.4e-13" iyy="3.13463693e-05" iyz="-2.8154088e-07" izz="1.91534236e-05"/>
+                <inertia ixx="4.41099235e-05" ixy="-0" ixz="-5.4e-13" iyy="3.13463693e-05" iyz="-2.8154088e-10" izz="1.91534236e-05"/>
             </inertial>
             <visual name="">
@@ -124,7 +124,7 @@
         <link name="${name}_foot">
             <inertial>
-                <origin xyz="0.0 0.0 0.0" rpy="0.0 0.0 0.0"/>
-                <mass value="1.0"/>
-                <inertia ixx="0.0" ixy="0.0" ixz="0.0" iyy="0.0" iyz="0.0" izz="0.0"/>
+                <origin xyz="0.0 -0.015 0.03" rpy="0.0 0.0 0.0"/>
+                <mass value="0.080"/>
+                <inertia ixx="0.000086666666666667" ixy="0.0" ixz="0.0" iyy="0.000104666666666667" iyz="0.0" izz="0.00003"/>
             </inertial>
             <visual name="">
@@ -136,10 +136,20 @@
             </visual>
             <collision>
-                <origin xyz="0.0 -0.04 0.04" rpy="0.0 0.0 0.0"/>
+                <origin xyz="0.0 -0.04 0.04" rpy="0.0 ${PI/2} 0.0"/>
                 <geometry>
-                    <box size="0.10 0.005 0.14"/>
+                    <!-- <box size="0.10 0.005 0.14"/> -->
+                    <mesh filename="package://automi_description/meshes/foot.stl"  scale="1e-2 1e-2 1e-2"/>
                 </geometry>
             </collision>
         </link>
+        <gazebo reference="${name}_foot">
+            <material>Gazebo/SkyBlue</material>
+            <mu1>9000</mu1>
+            <mu2>9000</mu2>
+            <kp>1000000.0</kp>
+            <kd>10.0</kd>
+            <minDepth>0.001</minDepth>
+            <maxContacts>1</maxContacts>
+        </gazebo>
     </xacro:macro>
 </robot>

File: automi_description/urdf/torso.urdf.xacro (robot description, xacro)
@@ -13,7 +13,7 @@
         <link name="${name}_hip">
             <inertial>
-                <origin xyz="0.0 0.0 0.0" rpy="0.0 0.0 0.0"/>
+                <origin xyz="0.0 0.0 0.0" rpy="${PI/2} 0.0 ${PI/2}"/>
                 <mass value="0.131665"/>
-                <inertia ixx="0.000519418268" ixy="-1.79595195e-05" ixz="1.2075507e-07" iyy="0.00048709882" iyz="3.8656764e-07" izz="0.000115698856"/>
+                <inertia ixx="0.000519418268" ixy="0" ixz="0" iyy="0.00048709882" iyz="0" izz="0.000115698856"/>
             </inertial>
             <visual>
@@ -43,7 +43,7 @@
         <link name="${name}_core">
             <inertial>
-                <origin xyz="0.0 0.0 0.0" rpy="0.0 0.0 0.0"/>
+                <origin xyz="0.0 0.0 0.01" rpy="${PI/2} 0.0 ${PI/2}"/>
                 <mass value="1.55086"/>
-                <inertia ixx="0.0034367683" ixy="5.09836432e-05" ixz="4.77030168e-06" iyy="0.00293127768" iyz="-4.57789663e-05" izz="0.00196796593"/>
+                <inertia ixx="0.0034367683" ixy="0" ixz="0" iyy="0.00293127768" iyz="0" izz="0.00196796593"/>
             </inertial>
             <visual name="">
@@ -73,5 +73,5 @@
         <link name="${name}_chest">
             <inertial>
-                <origin xyz="0.0 0.0 0.0" rpy="0.0 0.0 0.0"/>
+                <origin xyz="0.0 0.0 0.02" rpy="${PI/2} 0.0 ${PI/2}"/>
                 <mass value="0.128678"/>
                 <inertia ixx="0.000284733358" ixy="-1.04236092e-06" ixz="-7.3232262e-07" iyy="0.000360225319" iyz="-6.1818174e-07" izz="0.000135432051"/>
@@ -128,5 +128,5 @@
         <link name="${name}_camera_link">
             <inertial>
-                <origin xyz="0.0 0.0 0.0" rpy="0.0 0.0 0.0"/>
+                <origin xyz="-0.01 0.0 0.0" rpy="0.0 ${-PI/2} 0.0"/>
                 <mass value="0.0197099"/>
                 <inertia ixx="3.31024347e-06" ixy="-8.1e-13" ixz="-8.1e-13" iyy="8.74277118e-06" iyz="-4.4037e-10" izz="7.77454497e-06"/>
@@ -152,4 +152,9 @@
             </material>
         </gazebo>
+        <gazebo reference="${name}_core">
+            <material>
+                Gazebo/Orange
+            </material>
+        </gazebo>
     </xacro:macro>
 </robot>
