Commit message: adjusted leg.urdf.xacro

File: automi_description/urdf/automi.urdf.xacro (robot description, xacro)
@@ -3,6 +3,36 @@
     <xacro:property name="PI" value="3.1415926535897931"/>
     <xacro:include filename="$(find automi_description)/urdf/dynamixels.urdf.xacro" />
-    <xacro:include filename="$(find automi_description)/urdf/torso.urdf.xacro" />
-    <xacro:include filename="$(find automi_description)/urdf/arm.urdf.xacro" />
+    <!-- <xacro:include filename="$(find automi_description)/urdf/torso.urdf.xacro" /> -->
+    <!-- <xacro:include filename="$(find automi_description)/urdf/arm.urdf.xacro" /> -->
     <xacro:include filename="$(find automi_description)/urdf/leg.urdf.xacro" />
+    <link name="1">
+        <inertial>
+            <origin xyz="0.0 0.0 0.0" rpy="0.0 0.0 0.0"/>
+            <mass value="1.0"/>
+            <inertia ixx="0.0" ixy="0.0" ixz="0.0" iyy="0.0" iyz="0.0" izz="0.0"/>
+        </inertial>
+        <collision>
+            <origin xyz="0.0 0.0 0.0" rpy="0.0 0.0 0.0"/>
+            <geometry>
+                <box size="0.1 0.05 0.05"/>
+            </geometry>
+        </collision>
+        <visual>
+            <geometry>
+                <box size="0.1 0.05 0.05"/>
+            </geometry>
+        </visual>
+    </link>
+    <xacro:leg
+        name="left"
+        parent="1"
+        reflect="1">
+        <origin xyz="0.1 0.0 0.0" rpy="0.0 ${PI} 0.0"/>
+    </xacro:leg>
+    <xacro:leg
+        name="right"
+        parent="1"
+        reflect="-1">
+        <origin xyz="-0.1 0.0 0.0" rpy="0.0 ${PI} 0.0"/>
+    </xacro:leg>
 </robot>

File: automi_description/urdf/dynamixels.urdf.xacro (robot description, xacro)
@@ -1,16 +1,29 @@
 <?xml version="1.0"?>
 <robot xmlns:xacro="http://www.ros.org/wiki/xacro">
-    <xacro:macro name="AX12" params="name *origin parent child">
+    <xacro:macro name="AX12" params="name parent child *p_origin *c_origin">
+        <joint name="${name}" type="revolute">
+            <xacro:insert_block name="c_origin"/>
+            <parent link="${name}_AX12"/>
+            <child link ="${child}"/>
+            <axis xyz="0 0 1"/>
+            <limit
+                effort="150.0"
+                velocity="12.0"
+                lower="-2e16"
+                upper="2e16"/>
+        </joint>
+        <gazebo reference="${name}">
+			<provideFeedback>true</provideFeedback>
+            <preserveFixedJoint>true</preserveFixedJoint>
+		</gazebo>
         <joint name="${name}_dyn_fixed" type="fixed">
-            <xacro:insert_block name="origin"/>
+            <xacro:insert_block name="p_origin"/>
             <parent link="${parent}"/>
             <child link ="${name}_AX12"/>
         </joint>
-        <joint name="${name}" type="revolute">
-            <origin xyz="0 0 -0.01">
-            <parent link="${name}_AX12"/>
-            <child link ="${child}"/>
-            <axis xyz="1 0 0"/>
-        </joint>
+        <gazebo reference="${name}_dyn_fixed">
+			<provideFeedback>true</provideFeedback>
+            <preserveFixedJoint>true</preserveFixedJoint>
+		</gazebo>
         <link name="${name}_AX12">
             <inertial>
@@ -39,16 +52,29 @@
         </gazebo>
     </xacro:macro>
-    <xacro:macro name="MX28" params="name *origin parent child">
+    <xacro:macro name="MX28" params="name parent child *p_origin *c_origin">
+        <joint name="${name}" type="revolute">
+            <xacro:insert_block name="c_origin"/>
+            <parent link="${name}_MX28"/>
+            <child link ="${child}"/>
+            <axis xyz="0 0 1"/>
+            <limit
+                effort="150.0"
+                velocity="12.0"
+                lower="-2e16"
+                upper="2e16"/>
+        </joint>
+        <gazebo reference="${name}">
+			<provideFeedback>true</provideFeedback>
+            <preserveFixedJoint>true</preserveFixedJoint>
+		</gazebo>
         <joint name="${name}_dyn_fixed" type="fixed">
-            <xacro:insert_block name="origin"/>
+            <xacro:insert_block name="p_origin"/>
             <parent link="${parent}"/>
             <child link ="${name}_MX28"/>
         </joint>
-        <joint name="${name}" type="revolute">
-            <origin xyz="0 0 -0.01">
-            <parent link="${name}_MX28"/>
-            <child link ="${child}"/>
-            <axis xyz="1 0 0"/>
-        </joint>
+        <gazebo reference="${name}_dyn_fixed">
+			<provideFeedback>true</provideFeedback>
+            <preserveFixedJoint>true</preserveFixedJoint>
+		</gazebo>
         <link name="${name}_MX28">
             <inertial>
@@ -77,16 +103,29 @@
         </gazebo>
     </xacro:macro>
-    <xacro:macro name="MX64" params="name *origin parent child">
+    <xacro:macro name="MX64" params="name parent child *p_origin *c_origin">
+        <joint name="${name}" type="revolute">
+            <xacro:insert_block name="c_origin"/>
+            <parent link="${name}_MX64"/>
+            <child link ="${child}"/>
+            <axis xyz="0 0 1"/>
+            <limit
+                effort="150.0"
+                velocity="12.0"
+                lower="-2e16"
+                upper="2e16"/>
+        </joint>
+        <gazebo reference="${name}">
+			<provideFeedback>true</provideFeedback>
+            <preserveFixedJoint>true</preserveFixedJoint>
+		</gazebo>
         <joint name="${name}_dyn_fixed" type="fixed">
-            <xacro:insert_block name="origin"/>
+            <xacro:insert_block name="p_origin"/>
             <parent link="${parent}"/>
             <child link ="${name}_MX64"/>
         </joint>
-        <joint name="${name}" type="revolute">
-            <origin xyz="0 0 -0.01">
-            <parent link="${name}_MX64"/>
-            <child link ="${child}"/>
-            <axis xyz="1 0 0"/>
-        </joint>
+        <gazebo reference="${name}_dyn_fixed">
+			<provideFeedback>true</provideFeedback>
+            <preserveFixedJoint>true</preserveFixedJoint>
+		</gazebo>
         <link name="${name}_MX64">
             <inertial>

File: automi_description/urdf/leg.urdf.xacro (robot description, xacro)
@@ -2,37 +2,28 @@
 <robot xmlns:xacro="http://www.ros.org/wiki/xacro">
     <xacro:macro name="leg" params="name *origin parent reflect">
-        <!-- JOINTS -->
-        <joint name="${name}_fixed" type="fixed">
-            <xacro:insert_block name="origin"/>
-            <parent link="${parent}"/>
-            <child link="${name}"/>
-        </joint>
         <!-- LINKS -->
-        <link name="${name}">
-            <inertial>
-                <mass value="0.0"/>
-            </inertial>
-        </link>
         <xacro:AX12
             name="${name}_hip_yaw"
-            parent="${name}"
+            parent="${parent}"
             child="${name}_top_Ubar">
-            <origin xyz="0.0 0.0 0.0" rpy="0.0 ${PI/2} 0.0"/>
+            <xacro:insert_block name="origin"/>
+            <origin xyz="0.0 0.0 -0.01" rpy="0.0 0.0 0.0"/>
         </xacro:AX12>
         <link name="${name}_top_Ubar">
             <inertial>
                 <origin xyz="0.0 0.0 0.0" rpy="0.0 0.0 0.0"/>
-                <mass value="0.0"/>
+                <mass value="1.0"/>
                 <inertia ixx="0.0" ixy="0.0" ixz="0.0" iyy="0.0" iyz="0.0" izz="0.0"/>
             </inertial>
             <collision>
-                <origin xyz="0.0 0.0 0.0" rpy="0.0 0.0 0.0"/>
+                <origin xyz="0.0 0.0 0.04" rpy="0.0 0.0 ${PI/2}"/>
                 <geometry>
-                    <box size="0.0 0.0 0.0"/>
+                    <box size="0.15 0.05 0.005"/>
                 </geometry>
             </collision>
-            <visual>
+            <visual name="">
+                <origin xyz="0.0 0.0 0.04" rpy="0.0 0.0 ${PI/2}"/>
                 <geometry>
-                    <box size="0.0 0.0 0.0"/>
+                    <box size="0.15 0.05 0.005"/>
                 </geometry>
             </visual>
@@ -41,29 +32,38 @@
             name="${name}_hip_roll"
             parent="${name}_top_Ubar"
-            child="${name}_hip_pitch_MX64">
-            <origin xyz="0.0 0.0 0.0" rpy="0.0 0.0 0.0"/>
+            child="${name}_int_hip">
+            <origin xyz="0.0 0.03 0.07" rpy="${PI/2} 0.0 0.0"/>
+            <origin xyz="0.0 0.0 0.05" rpy="0 0 0.0"/>
         </xacro:MX28>
+        <link name="${name}_int_hip">
+            <inertial>
+                <origin xyz="0.0 0.0 0.0" rpy="0.0 0.0 0.0"/>
+                <mass value="0.0005"/>
+                <inertia ixx="0.0" ixy="0.0" ixz="0.0" iyy="0.0" iyz="0.0" izz="0.0"/>
+            </inertial>
+        </link>
         <xacro:MX64
             name="${name}_hip_pitch"
-            parent="${name}_hip_roll_MX28"
+            parent="${name}_int_hip"
             child="${name}_upper_leg">
-            <origin xyz="0.0 0.0 0.0" rpy="0.0 0.0 ${PI/2}"/>
+            <origin xyz="0.0 0.0 0.0" rpy="0.0 0.0 0.0"/>
+            <origin xyz="0.0 0.0 0.0" rpy="${PI/2} 0.0 ${PI/2}"/>
         </xacro:MX64>
         <link name="${name}_upper_leg">
             <inertial>
                 <origin xyz="0.0 0.0 0.0" rpy="0.0 0.0 0.0"/>
-                <mass value="0.0"/>
+                <mass value="1.0"/>
                 <inertia ixx="0.0" ixy="0.0" ixz="0.0" iyy="0.0" iyz="0.0" izz="0.0"/>
             </inertial>
-            <visual>
-                <origin xyz="0.0 0.0 0.0" rpy="0.0 0.0 0.0"/>
+            <visual name="">
+                <origin xyz="0.075 0.0 0.0" rpy="0.0 0.0 0.0"/>
                 <geometry>
-                    <box size="0.03 0.03 0.10"/>
+                    <box size="0.15 0.025 0.025"/>
                 </geometry>
             </visual>
             <collision>
-                <origin xyz="0.0 0.0 0.0" rpy="0.0 0.0 0.0"/>
+                <origin xyz="0.075 0.0 0.0" rpy="0.0 0.0 0.0"/>
                 <geometry>
-                    <box size="0.03 0.03 0.10"/>
+                    <box size="0.15 0.025 0.025"/>
                 </geometry>
             </collision>
@@ -73,10 +73,51 @@
             parent="${name}_upper_leg"
             child="${name}_lower_leg">
-            <origin xyz="0.0 0.0 0.0" rpy="0.0 ${PI} ${PI/2}"/>
+            <origin xyz="0.15 0.0 0.0" rpy="0.0 0.0 ${PI/2}"/>
+            <origin xyz="0.0 0.0 0.0" rpy="0.0 0.0 0.0"/>
         </xacro:MX28>
         <link name="${name}_lower_leg">
             <inertial>
                 <origin xyz="0.0 0.0 0.0" rpy="0.0 0.0 0.0"/>
-                <mass value="0.0"/>
+                <mass value="1.0"/>
+                <inertia ixx="0.0" ixy="0.0" ixz="0.0" iyy="0.0" iyz="0.0" izz="0.0"/>
+            </inertial>
+            <visual name="">
+                <origin xyz="0.0 -0.075 0.0" rpy="0.0 0.0 0.0"/>
+                <geometry>
+                    <box size="0.025 0.15 0.025"/>
+                </geometry>
+            </visual>
+            <collision>
+                <origin xyz="0.0 -0.075 0.0" rpy="0.0 0.0 0.0"/>
+                <geometry>
+                    <box size="0.025 0.15 0.025"/>
+                </geometry>
+            </collision>
+        </link>
+        <xacro:MX28
+            name="${name}_ankle_pitch"
+            parent="${name}_lower_leg"
+            child="${name}_int_ankle">
+            <origin xyz="0.0 -0.15 0.0" rpy="0.0 ${PI} 0"/>
+            <origin xyz="0.0 0.0 0.0" rpy="0.0 0.0 0.0"/>
+        </xacro:MX28>
+        <link name="${name}_int_ankle">
+            <inertial>
+                <origin xyz="0.0 0.0 0.0" rpy="0.0 0.0 0.0"/>
+                <mass value="0.0005"/>
+                <inertia ixx="0.0" ixy="0.0" ixz="0.0" iyy="0.0" iyz="0.0" izz="0.0"/>
+            </inertial>
+        </link>
+        <xacro:MX64
+            name="${name}_ankle_roll"
+            parent="${name}_int_ankle"
+            child="${name}_foot">
+            <origin xyz="0.05 0.0 0.0" rpy="0 0 0"/>
+            <origin xyz="-0.03 -0.03 0.0" rpy="0 ${PI/2} 0.0"/>
+        </xacro:MX64>
+        <link name="${name}_foot">
+            <inertial>
+                <origin xyz="0.0 0.0 0.0" rpy="0.0 0.0 0.0"/>
+                <mass value="1.0"/>
                 <inertia ixx="0.0" ixy="0.0" ixz="0.0" iyy="0.0" iyz="0.0" izz="0.0"/>
             </inertial>
@@ -84,5 +125,5 @@
                 <origin xyz="0.0 0.0 0.0" rpy="0.0 0.0 0.0"/>
                 <geometry>
-                    <box size="0.03 0.03 0.10"/>
+                    <box size="0.10 0.005 0.14"/>
                 </geometry>
             </visual>
@@ -90,38 +131,8 @@
                 <origin xyz="0.0 0.0 0.0" rpy="0.0 0.0 0.0"/>
                 <geometry>
-                    <box size="0.03 0.03 0.10"/>
+                    <box size="0.10 0.005 0.14"/>
                 </geometry>
             </collision>
         </link>
-        <xacro:MX28
-            name="${name}_angle_pitch"
-            parent="${name}_lower_leg"
-            child="${name}_angle_roll_MX64">
-            <origin xyz="0.0 0.0 0.0" rpy="0.0 ${PI} ${PI/2}"/>
-        </xacro:MX28>
-        <xacro:MX64
-            name="${name}_angle_roll"
-            parent="${name}_angle_pitch_MX28"
-            child="${name}_foot">
-            <origin xyz="0.0 0.0 0.0" rpy="${PI} 0.0 0"/>
-        </xacro:MX64>
-        <link name="${name}_foot">
-            <inertial>
-                <origin xyz="0.0 0.0 0.0" rpy="0.0 0.0 0.0"/>
-                <mass value="0.0"/>
-                <inertia ixx="0.0" ixy="0.0" ixz="0.0" iyy="0.0" iyz="0.0" izz="0.0"/>
-            </inertial>
-            <visual name="">
-                <origin xyz="0.0 0.0 0.0" rpy="0.0 0.0 0.0"/>
-                <geometry>
-                    <box size="0.05 0.07 0.005"/>
-                </geometry>
-            </visual>
-            <collision>
-                <origin xyz="0.0 0.0 0.0" rpy="0.0 0.0 0.0"/>
-                <geometry>
-                    <box size="0.05 0.07 0.005"/>
-                </geometry>
-            </collision>
-        </link>
+    </xacro:macro>
 </robot>

Commit message: added controllers

File: automi_description/urdf/automi.urdf.xacro (robot description, xacro)
@@ -9,4 +9,5 @@
         <inertial>
             <mass value="0.0005"/>
+            <inertia ixx="0.0" ixy="0.0" ixz="0.0" iyy="0.0" iyz="0.0" izz="0.0"/>
         </inertial>
     </link>
@@ -41,41 +42,18 @@
     </xacro:arm>
     <gazebo>
-        <plugin name="joint_state_publisher" filename="libgazebo_ros_joint_state_publisher.so">
-            <jointName>
-                head_pan    ,
-                head_tilt   ,
-                r_hip_r     ,
-                r_hip_p     ,
-                r_hip_y     ,
-                r_knee      ,
-                r_ankle_r   ,
-                r_ankle_p   ,
-                r_shoulder_r,
-                r_shoulder_p,
-                r_elbow     ,
-                l_hip_r     ,
-                l_hip_p     ,
-                l_hip_y     ,
-                l_knee      ,
-                l_ankle_r   ,
-                l_ankle_p   ,
-                l_shoulder_r,
-                l_shoulder_p,
-                l_elbow
-            </jointName>
-            <updateRate>60.0</updateRate>
-            <alwaysOn>true</alwaysOn>
+        <plugin filename="libgazebo_ros_control.so" name="gazebo_ros_control">
+            <robotNamespace>/automi</robotNamespace>
         </plugin>
     </gazebo>
     <xacro:macro name="trans" params="num joint">
         <transmission name="tran${num}">
-        <joint name="${joint}">
-            <hardwareInterface>hardware_interface/PositionJointInterface</hardwareInterface>
-        </joint>
-        <type>transmission_interface/SimpleTransmission</type>
-        <actuator name="servo${num}">
-            <hardwareInterface>hardware_interface/PositionJointInterface</hardwareInterface>
-            <mechanicalReduction>1</mechanicalReduction>
-        </actuator>
+            <joint name="${joint}">
+                <hardwareInterface>hardware_interface/PositionJointInterface</hardwareInterface>
+            </joint>
+            <type>transmission_interface/SimpleTransmission</type>
+            <actuator name="servo${num}">
+                <hardwareInterface>hardware_interface/PositionJointInterface</hardwareInterface>
+                <mechanicalReduction>1</mechanicalReduction>
+            </actuator>
         </transmission>
     </xacro:macro>

File: automi_description/urdf/torso.urdf.xacro (robot description, xacro)
@@ -95,4 +95,5 @@
             <inertial>
                 <mass value="0.0005"/>
+                <inertia ixx="0.0" ixy="0.0" ixz="0.0" iyy="0.0" iyz="0.0" izz="0.0"/>
             </inertial>
         </link>

Commit message: fixed leg oscillations

File: automi_description/urdf/automi.urdf.xacro (robot description, xacro)
@@ -6,4 +6,5 @@
     <xacro:include filename="$(find automi_description)/urdf/arm.urdf.xacro" />
     <xacro:include filename="$(find automi_description)/urdf/leg.urdf.xacro" />
+    <xacro:include filename="$(find automi_description)/urdf/transmissions.urdf.xacro" />
     <link name="floating_base">
         <inertial>
@@ -46,35 +47,3 @@
         </plugin>
     </gazebo>
-    <xacro:macro name="trans" params="num joint">
-        <transmission name="tran${num}">
-            <joint name="${joint}">
-                <hardwareInterface>hardware_interface/PositionJointInterface</hardwareInterface>
-            </joint>
-            <type>transmission_interface/SimpleTransmission</type>
-            <actuator name="servo${num}">
-                <hardwareInterface>hardware_interface/PositionJointInterface</hardwareInterface>
-                <mechanicalReduction>1</mechanicalReduction>
-            </actuator>
-        </transmission>
-    </xacro:macro>
-    <xacro:trans num="1"  joint="r_hip_r"/>
-    <xacro:trans num="2"  joint="r_hip_p"/>
-    <xacro:trans num="3"  joint="r_hip_y"/>
-    <xacro:trans num="4"  joint="r_knee"/>
-    <xacro:trans num="5"  joint="r_ankle_r"/>
-    <xacro:trans num="6"  joint="r_ankle_p"/>
-    <xacro:trans num="7" joint="l_hip_r"/>
-    <xacro:trans num="8" joint="l_hip_p"/>
-    <xacro:trans num="9" joint="l_hip_y"/>
-    <xacro:trans num="10" joint="l_knee"/>
-    <xacro:trans num="11" joint="l_ankle_r"/>
-    <xacro:trans num="12" joint="l_ankle_p"/>
-    <xacro:trans num="13"  joint="r_shoulder_r"/>
-    <xacro:trans num="14" joint="r_shoulder_p"/>
-    <xacro:trans num="15" joint="r_elbow"/>
-    <xacro:trans num="16" joint="l_shoulder_r"/>
-    <xacro:trans num="17" joint="l_shoulder_p"/>
-    <xacro:trans num="18" joint="l_elbow"/>
-    <xacro:trans num="19"  joint="head_pan"/>
-    <xacro:trans num="20"  joint="head_tilt"/>
 </robot>

File: automi_description/urdf/leg.urdf.xacro (robot description, xacro)
@@ -143,12 +143,27 @@
             </collision>
         </link>
+        <joint name="${name}_foot_base_j" type="fixed">
+            <origin xyz="0.0 0.0 0.0" rpy="0.0 0.0 0.0"/>
+            <parent link="${name}_foot"/>
+            <child link="${name}_foot_base"/>
+        </joint>
+        <link name="${name}_foot_base">
+            <collision>
+                <origin xyz="0.0 -0.04 0.03" rpy="0.0 0.0 0.0"/>
+                <geometry>
+                    <box size="0.08 0.005 0.12"/>
+                </geometry>
+            </collision>
+        </link>
         <gazebo reference="${name}_foot">
             <material>Gazebo/SkyBlue</material>
-            <mu1>9000</mu1>
-            <mu2>9000</mu2>
-            <kp>1000000.0</kp>
-            <kd>10.0</kd>
+        </gazebo>
+        <gazebo reference="${name}_foot_base">
+            <mu1>1</mu1>
+            <mu2>1</mu2>
+            <kp>0.0</kp>
+            <kd>10000.0</kd>
             <minDepth>0.001</minDepth>
-            <maxContacts>1</maxContacts>
+            <maxContacts>2</maxContacts>
         </gazebo>
     </xacro:macro>
